File: Battery-SegmentPCB-A/Battery-SegmentPCB-A.kicad_pcb (KiCad board)
At the start: 2 copper layers, 556.2 x 27.7 mm, 20 parts, among them J1 Conn_01x04, J10 Conn_01x16, J11 Conn_01x09, J2 Conn_01x04, J3 Conn_01x04, J4 Conn_01x04, J5 Conn_01x04, J6 Conn_01x04, J7 Conn_01x04, J8 Conn_01x04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

Commit message: updated boards
Parts:
- removed the J1 at (576.0, 128.1)
- removed J10: Conn_01x16, footprints:CON_430451612_MOL
- removed the J2 at (562.3, 128.1)
- removed the J3 at (431.4, 128.1)
- removed the J4 at (417.6, 128.1)
- removed the J5 at (286.7, 128.1)
- removed the J6 at (272.9, 128.1)
- removed the J7 at (142.1, 128.1)
- removed the J8 at (128.1, 128.1)
- removed the J9 at (541.8, 127.9)
- J1, J2, J3, J4, J5, J6, J7, J8: moved to B.Cu
- moved J4 286.0 mm to (601.5, 124.0), turned to 180 degrees
- moved J3 270.7 mm to (588.0, 124.0), turned to 180 degrees
- moved J2 232.4 mm to (551.0, 124.0), turned to 180 degrees
- moved J1 217.9 mm to (538.0, 124.0), turned to 180 degrees
- moved J5 207.9 mm to (126.5, 127.2), turned to 180 degrees
- moved J6 198.4 mm to (140.7, 127.2), turned to 180 degrees
- moved J9 113.2 mm to (463.7, 112.0)
- moved J11 110.9 mm to (463.2, 126.0)
- moved J8 107.3 mm to (285.7, 126.2), turned to 180 degrees
- moved J7 103.8 mm to (272.5, 126.0), turned to 180 degrees
Routing:
- net /TEMP_5: track 0.00 -> 337.6 mm
- net /VOLT1_5 +: track 0.00 -> 331.5 mm
- net /TEMP_6: track 0.00 -> 320.8 mm
- net /VOLT1_6 +: track 0.00 -> 312.5 mm
- net /TEMP_7: track 0.00 -> 185.5 mm
- net /VOLT1_7 +: track 0.00 -> 178.9 mm
- net /TEMP_8: track 0.00 -> 165.0 mm
- net /VOLT1_8 +: track 0.00 -> 160.4 mm
- net /TEMP_4: track 0.00 -> 153.2 mm
- net /VOLT1_4 +: track 0.00 -> 147.8 mm
- net /TEMP_3: track 0.00 -> 143.1 mm
- net /VOLT1_3 +: track 0.00 -> 129.9 mm
- net /TEMP_2: track 0.00 -> 94.1 mm
- net /VOLT1_2 +: track 0.00 -> 89.5 mm
- net /TEMP_1: track 0.00 -> 77.2 mm
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- added copper zone on B.Cu, net /TEMP_GND
- removed copper zone on F.Cu, net (none)
Other:
- outline, holes or cut-outs redrawn
