File: Battery-SegmentPCB-A/Battery-SegmentPCB-A.kicad_pcb (KiCad board)
At the start: 2 copper layers, 556.2 x 27.7 mm, 20 parts, among them J1 Conn_01x04, J10 Conn_01x16, J11 Conn_01x09, J2 Conn_01x04, J3 Conn_01x04, J4 Conn_01x04, J5 Conn_01x04, J6 Conn_01x04, J7 Conn_01x04, J8 Conn_01x04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

Commit message: new template
Parts:
- removed J1 (x2), J2 (x2), J3 (x2), J4 (x2), J5 (x2), J6 (x2), J7 (x2), J8 (x2): Conn_01x04, footprints:CONN_S4B-PH-K-S_JST
- removed J10: Conn_01x16, footprints:CON_430451612_MOL
- removed J11, J9 (x2): Conn_01x09, footprints:CON_436500915_MOL
Routing:
- removed copper zone on F.Cu, net (none)
Other:
- board size 556.2 x 27.7 mm -> 522.7 x 21.7 mm

Commit message: started
Parts:
- added J1: Conn_01x01, MountingHole:MountingHole_3.2mm_M3_DIN965_Pad_TopOnly, F.Cu at (601.7, 113.4)
- added J10: Conn_01x09, footprints:CON_436500915_MOL, F.Cu at (434.0, 119.2)
- added J11: Conn_01x01, MountingHole:MountingHole_3.2mm_M3_DIN965_Pad_TopOnly, F.Cu at (314.5, 113.4)
- added J12: Conn_01x01, MountingHole:MountingHole_3.2mm_M3_DIN965_Pad_TopOnly, F.Cu at (314.5, 127.6)
- added J13: Conn_01x01, MountingHole:MountingHole_3.2mm_M3_DIN965_Pad_TopOnly, F.Cu at (242.6, 113.4)
- added J14: Conn_01x01, MountingHole:MountingHole_3.2mm_M3_DIN965_Pad_TopOnly, F.Cu at (242.6, 127.6)
- added J15: Conn_01x01, MountingHole:MountingHole_3.2mm_M3_DIN965_Pad_TopOnly, F.Cu at (170.8, 113.4)
- added J16: Conn_01x01, MountingHole:MountingHole_3.2mm_M3_DIN965_Pad_TopOnly, F.Cu at (170.8, 127.6)
- added J17: Conn_01x01, MountingHole:MountingHole_3.2mm_M3_DIN965_Pad_TopOnly, F.Cu at (99.0, 113.4)
- added J18: Conn_01x01, MountingHole:MountingHole_3.2mm_M3_DIN965_Pad_TopOnly, F.Cu at (99.0, 127.6)
- added J19: Conn_01x02, Connector_Molex:Molex_Nano-Fit_105309-xx02_1x02_P2.50mm_Vertical, F.Cu at (608.8, 118.5)
- added J2: Conn_01x01, MountingHole:MountingHole_3.2mm_M3_DIN965_Pad_TopOnly, F.Cu at (601.7, 127.6)
- added J20: Conn_01x02, Connector_Molex:Molex_Nano-Fit_105309-xx02_1x02_P2.50mm_Vertical, F.Cu at (539.3, 118.5)
- added J21: Conn_01x02, Connector_Molex:Molex_Nano-Fit_105309-xx02_1x02_P2.50mm_Vertical, F.Cu at (469.8, 118.5)
- added J22: Conn_01x02, Connector_Molex:Molex_Nano-Fit_105309-xx02_1x02_P2.50mm_Vertical, F.Cu at (400.3, 118.5)
- added J23: Conn_01x02, Connector_Molex:Molex_Nano-Fit_105309-xx02_1x02_P2.50mm_Vertical, F.Cu at (330.8, 118.5)
- added J24: Conn_01x02, Connector_Molex:Molex_Nano-Fit_105309-xx02_1x02_P2.50mm_Vertical, F.Cu at (261.2, 118.5)
- added J25: Conn_01x02, Connector_Molex:Molex_Nano-Fit_105309-xx02_1x02_P2.50mm_Vertical, F.Cu at (191.7, 118.5)
- added J26: Conn_01x02, Connector_Molex:Molex_Nano-Fit_105309-xx02_1x02_P2.50mm_Vertical, F.Cu at (122.2, 118.5)
- added J3: Conn_01x01, MountingHole:MountingHole_3.2mm_M3_DIN965_Pad_TopOnly, F.Cu at (529.9, 113.4)
- added J4: Conn_01x01, MountingHole:MountingHole_3.2mm_M3_DIN965_Pad_TopOnly, F.Cu at (529.9, 127.6)
- added J5: Conn_01x01, MountingHole:MountingHole_3.2mm_M3_DIN965_Pad_TopOnly, F.Cu at (458.1, 113.4)
- added J6: Conn_01x01, MountingHole:MountingHole_3.2mm_M3_DIN965_Pad_TopOnly, F.Cu at (458.1, 127.6)
- added J7: Conn_01x01, MountingHole:MountingHole_3.2mm_M3_DIN965_Pad_TopOnly, F.Cu at (386.3, 113.4)
- added J8: Conn_01x01, MountingHole:MountingHole_3.2mm_M3_DIN965_Pad_TopOnly, F.Cu at (386.3, 127.6)
- added J9: Conn_01x09, footprints:CON_436500915_MOL, F.Cu at (371.2, 119.2)
Other:
- board size 522.7 x 21.7 mm -> 522.7 x 21 mm

Commit message: womp womp(done)
Routing:
- net /TEMP_GND: track 0.00 -> 493.4 mm
- net /VOLT1_8 +: track 0.00 -> 314.5 mm
- net /VOLT1_7 +: track 0.00 -> 245.7 mm
- net /TEMP_1: track 0.00 -> 239.9 mm
- net /TEMP_8: track 0.00 -> 236.1 mm
- net /TEMP_7: track 0.00 -> 181.3 mm
- net /VOLT1_6 +: track 0.00 -> 176.9 mm
- net /VOLT1_1 +: track 0.00 -> 174.2 mm
- net /TEMP_2: track 0.00 -> 174.2 mm
- net /VOLT_1 -: track 0.00 -> 170.1 mm
- net /VOLT1_5 +: track 0.00 -> 108.0 mm
- net /TEMP_3: track 0.00 -> 107.7 mm
- net /TEMP_6: track 0.00 -> 106.9 mm
- net /VOLT1_2 +: track 0.00 -> 105.4 mm
- net /VOLT1_4 +: track 0.00 -> 40.8 mm
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Other:
- board text added: "-"
- board text added: "1"
- board text added: "1+"
- board text added: "1-"
- board text added: "2"
- board text added: "2+"
- board text added: "2-"
- board text added: "3"
- board text added: "3+"
- board text added: "3-"
- board text added: "4"
- board text added: "4+"
- board text added: "4-"
- board text added: "5"
- board text added: "5+"
- board text added: "5-"
- board text added: "6"
- board text added: "6+"
- board text added: "6-"
- board text added: "7"
- board text added: "7+"
- board text added: "7-"
- board text added: "8"
- board text added: "8+"
- board text added: "8-"
- board text added: "Temperature Connector"
- board text added: "Voltage Connector"

Commit message: b done
Routing:
- net /TEMP_GND: track 493.4 -> 0.00 mm
- net /VOLT1_8 +: track 314.5 -> 0.00 mm
- net /VOLT1_7 +: track 245.7 -> 0.00 mm
- net /TEMP_1: track 239.9 -> 0.00 mm
- net /TEMP_8: track 236.1 -> 0.00 mm
- net /TEMP_7: track 181.3 -> 0.00 mm
- net /VOLT1_6 +: track 176.9 -> 0.00 mm
- net /VOLT1_1 +: track 174.2 -> 0.00 mm
- net /TEMP_2: track 174.2 -> 0.00 mm
- net /VOLT_1 -: track 170.1 -> 0.00 mm
- net /VOLT1_5 +: track 108.0 -> 0.00 mm
- net /TEMP_3: track 107.7 -> 0.00 mm
- net /TEMP_6: track 106.9 -> 0.00 mm
- net /VOLT1_2 +: track 105.4 -> 0.00 mm
- net /VOLT1_4 +: track 40.8 -> 0.00 mm
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
Commit message: stuff
Parts:
- added F37: PTC Fuse, footprints:FUSC1810X100N, B.Cu at (596.9, 115.7)
- added F38: PTC Fuse, footprints:FUSC1810X100N, B.Cu at (524.9, 129.4)
- added F39: PTC Fuse, footprints:FUSC1810X100N, B.Cu at (463.4, 115.7)
- added F40: PTC Fuse, footprints:FUSC1810X100N, B.Cu at (391.1, 129.6)
- added F41: PTC Fuse, footprints:FUSC1810X100N, B.Cu at (316.4, 117.7)
- added F42: PTC Fuse, footprints:FUSC1810X100N, B.Cu at (247.0, 129.8)
- added F43: PTC Fuse, footprints:FUSC1810X100N, B.Cu at (174.1, 117.9)
- added F44: PTC Fuse, footprints:FUSC1810X100N, B.Cu at (105.0, 129.0)
- added G***: LHRs_LOGO, UTSVT_Logos:LHRs_LOGO, F.Cu at (121.8, 128.7)
- J1, J11, J12, J13, J14, J15, J16, J17, J18, J2, J3, J4, J5, J6, J7, J8: moved to B.Cu
- J19, J20, J21, J22, J23, J24, J25, J26: footprint Connector_Molex:Molex_Nano-Fit_105309-xx02_1x02_P2.50mm_Vertical -> UTSVT_Connectors:105313-2102
- moved J9 113.6 mm to (484.6, 125.9), turned to 180 degrees
- moved J10 74.8 mm to (508.7, 115.7)
- moved J21 21.7 mm to (449.0, 112.2), turned to -90 degrees
- moved J19 18.4 mm to (591.8, 111.6), turned to -90 degrees
- moved J26 14.7 mm to (109.4, 111.2), turned to -90 degrees
- moved J1 14.1 mm to (601.7, 127.6)
- moved J11 14.1 mm to (314.5, 127.6)
- moved J12 14.1 mm to (314.5, 113.4)
- moved J15 14.1 mm to (170.8, 127.6)
- moved J16 14.1 mm to (170.8, 113.4)
- moved J2 14.1 mm to (601.7, 113.4)
- moved J5 14.1 mm to (458.1, 127.6)
- moved J6 14.1 mm to (458.1, 113.4)
- moved J25 12.2 mm to (181.8, 111.6), turned to -90 degrees
- moved J24 10.0 mm to (254.1, 111.6), turned to -90 degrees
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Connections:
- J12 pad 1: /VOLT1_5 + -> Net-(J12-Pin_1)
- J14 pad 1: /VOLT1_6 + -> Net-(J14-Pin_1)
- J16 pad 1: /VOLT1_7 + -> Net-(J16-Pin_1)
- J18 pad 1: /VOLT1_8 + -> Net-(J18-Pin_1)
- J2 pad 1: /VOLT1_1 + -> Net-(J2-Pin_1)
- J4 pad 1: /VOLT1_2 + -> Net-(J4-Pin_1)
- J6 pad 1: /VOLT1_3 + -> Net-(J6-Pin_1)
- J8 pad 1: /VOLT1_4 + -> Net-(J8-Pin_1)
Routing:
- net /TEMP_GND: track 0.00 -> 514.2 mm, vias 0 -> 1
- net /VOLT1_8 +: track 0.00 -> 387.3 mm, vias 0 -> 1
- net /VOLT1_7 +: track 0.00 -> 324.3 mm, vias 0 -> 1
- net /VOLT1_6 +: track 0.00 -> 254.0 mm, vias 0 -> 1
- net /VOLT1_5 +: track 0.00 -> 184.9 mm, vias 0 -> 1
- net /TEMP_1: track 0.00 -> 128.6 mm, vias 0 -> 1
- net /VOLT1_4 +: track 0.00 -> 114.7 mm, vias 0 -> 1
- net /VOLT1_1 +: track 0.00 -> 111.8 mm, vias 0 -> 2
- net /TEMP_4: track 0.00 -> 108.3 mm, vias 0 -> 1
- net /TEMP_2: track 0.00 -> 74.0 mm, vias 0 -> 1
- net /TEMP_3: track 0.00 -> 52.4 mm, vias 0 -> 1
- net /VOLT1_3 +: track 0.00 -> 36.2 mm
- net /VOLT1_2 +: track 0.00 -> 31.8 mm, vias 0 -> 2
- net Net-(J18-Pin_1): track 0.00 -> 5.56 mm
- net Net-(J16-Pin_1): track 0.00 -> 5.39 mm
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Other:
- board text added: "Battery A Segment Day Fixed"
- board text added: "Battery B Segment Day Fixed"

Commit message: done?
Parts:
- moved J26 0.52 mm to (109.4, 111.8)
- moved J24 0.29 mm to (254.1, 111.8)
- moved J25 0.29 mm to (181.8, 111.8)
Routing:
- net /TEMP_8: track 0.00 -> 407.9 mm, vias 0 -> 2
- net /TEMP_7: track 0.00 -> 335.4 mm, vias 0 -> 3
- net /TEMP_6: track 0.00 -> 267.0 mm, vias 0 -> 3
- net /TEMP_5: track 0.00 -> 190.1 mm, vias 0 -> 2
- net /VOLT_1 -: track 0.04 -> 102.7 mm, vias 0 -> 1
- net /TEMP_2: track 74.0 -> 75.1 mm
Other:
- outline, holes or cut-outs redrawn
- board text removed: "Battery B Segment Day Fixed"

Commit message: seg A, 4 layer, moved conns, flipped fuses, fixed labels
Parts:
- F37, F38, F39, F40, F41, F42, F43, F44: moved to F.Cu
- moved F44 8.45 mm to (99.0, 123.0)
- moved F40 8.43 mm to (386.5, 122.5)
- moved F38 8.15 mm to (530.0, 123.0)
- moved F42 7.88 mm to (243.0, 123.0)
- moved F39 5.39 mm to (458.5, 118.0)
- moved F37 4.97 mm to (601.5, 117.5)
- moved F43 3.12 mm to (171.0, 117.5)
- moved F41 2.53 mm to (314.0, 118.5)
- moved J9 1.43 mm to (484.6, 124.5)
- moved J10 1.28 mm to (508.8, 117.0)
Connections:
- net /VOLT1_1 + renamed /VOLT_1 +
- net /VOLT1_2 + renamed /VOLT_2 +
- net /VOLT1_3 + renamed /VOLT_3 +
- net /VOLT1_4 + renamed /VOLT_4 +
- net /VOLT1_5 + renamed /VOLT_5 +
- net /VOLT1_6 + renamed /VOLT_6 +
- net /VOLT1_7 + renamed /VOLT_7 +
- net /VOLT1_8 + renamed /VOLT_8 +
Routing:
- net /TEMP_GND: track 514.0 -> 0.00 mm, vias 1 -> 0
- net /TEMP_8: track 407.9 -> 0.00 mm, vias 2 -> 0
- net /VOLT_8 +: track 387.3 -> 0.00 mm, vias 1 -> 0
- net /TEMP_7: track 335.4 -> 0.00 mm, vias 3 -> 0
- net /VOLT_7 +: track 324.3 -> 0.00 mm, vias 1 -> 0
- net /TEMP_6: track 267.0 -> 0.00 mm, vias 3 -> 0
- net /VOLT_6 +: track 254.0 -> 0.00 mm, vias 1 -> 0
- net /TEMP_5: track 190.1 -> 0.00 mm, vias 2 -> 0
- net /TEMP_1: track 128.6 -> 0.00 mm, vias 1 -> 0
- net /TEMP_4: track 108.3 -> 0.00 mm, vias 1 -> 0
- net /VOLT_1 -: track 102.7 -> 0.00 mm, vias 1 -> 0
- net /TEMP_2: track 75.1 -> 0.00 mm, vias 1 -> 0
- net /TEMP_3: track 52.4 -> 0.00 mm, vias 1 -> 0
- net /VOLT_1 +: track 111.8 -> 95.8 mm, vias 2 -> 0
- net Net-(J18-Pin_1): track 5.56 -> 0.00 mm
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- added copper zone on B.Cu, net /TEMP_GND
- added copper zone on In2.Cu, net /TEMP_GND
- added copper zone on F.Cu, net /VOLT_1 -
- added copper zone on In1.Cu, net /VOLT_1 -
Other:
- copper layers 2 -> 4
