File: Battery-SegmentPCB-A/Battery-SegmentPCB-A.kicad_pcb (KiCad board)
At the start: 4 copper layers, 522.7 x 21 mm, 35 parts, among them J1 Conn_01x01, J10 Conn_01x09, J11 Conn_01x01, J12 Conn_01x01, J13 Conn_01x01, J14 Conn_01x01, J15 Conn_01x01, J16 Conn_01x01, J17 Conn_01x01, J18 Conn_01x01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

Commit message: removed traces
Routing:
- net /VOLT_5 +: track 181.7 -> 0.00 mm
- net /VOLT_4 +: track 111.5 -> 0.00 mm
- net /VOLT_1 +: track 95.8 -> 0.00 mm
- net /VOLT_3 +: track 41.5 -> 0.00 mm
- net /VOLT_2 +: track 28.7 -> 0.00 mm
- net Net-(J12-Pin_1): track 5.67 -> 0.00 mm
- net Net-(J8-Pin_1): track 5.39 -> 0.00 mm
- net Net-(J4-Pin_1): track 5.02 -> 0.00 mm
- net Net-(J6-Pin_1): track 4.82 -> 0.00 mm
- net Net-(J2-Pin_1): track 4.38 -> 0.00 mm
Changed lines of the file:
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@@
 		)
-	)
-	(segment
-		(start 602.5 114.1912)
-		(end 601.74 113.4312)
-		(width 0.2)
-		(layer "F.Cu")
-		(net 18)
-	)
-	(segment
-		(start 602.5 117.5)
-		(end 602.5 114.1912)
-		(width 0.2)
-		(layer "F.Cu")
-		(net 18)
-	)
-	(segment
-		(start 531 123)
-		(end 531 123.5)
-		(width 0.2)
-		(layer "F.Cu")
-		(net 19)
-	)
-	(segment
-		(start 529.92 124.58)
-		(end 529.92 127.5687)
-		(width 0.2)
-		(layer "F.Cu")
-		(net 19)
-	)
-	(segment
-		(start 531 123.5)
-		(end 529.92 124.58)
-		(width 0.2)
-		(layer "F.Cu")
-		(net 19)
-	)
-	(segment
-		(start 458.1 117.4)
-		(end 457.5 118)
-		(width 0.2)
-		(layer "F.Cu")
-		(net 20)
-	)
-	(segment
-		(start 458.1 113.4312)
-		(end 458.1 117.4)
-		(width 0.2)
-		(layer "F.Cu")
-		(net 20)
-	)
-	(segment
-		(start 385.5 122.5)
-		(end 385.5 126.7887)
-		(width 0.2)
-		(layer "F.Cu")
-		(net 21)
-	)
-	(segment
-		(start 385.5 126.7887)
-		(end 386.28 127.5687)
-		(width 0.2)
-		(layer "F.Cu")
-		(net 21)
-	)
-	(segment
-		(start 313 118.5)
-		(end 313 114.8912)
-		(width 0.2)
-		(layer "F.Cu")
-		(net 22)
-	)
-	(segment
-		(start 313 114.8912)
-		(end 314.46 113.4312)
-		(width 0.2)
-		(layer "F.Cu")
-		(net 22)
-	)
-	(segment
-		(start 598.939 115.939)
-		(end 506.811001 115.939)
-		(width 0.2)
-		(layer "F.Cu")
-		(net 26)
-	)
-	(segment
-		(start 600.5 117.5)
-		(end 598.939 115.939)
-		(width 0.2)
-		(layer "F.Cu")
-		(net 26)
-	)
-	(segment
-		(start 506.811001 115.939)
-		(end 505.750001 117)
-		(width 0.2)
-		(layer "F.Cu")
-		(net 26)
-	)
-	(segment
-		(start 529 123)
-		(end 514.395584 123)
-		(width 0.2)
-		(layer "F.Cu")
-		(net 27)
-	)
-	(segment
-		(start 509.456584 118.061)
-		(end 503.811002 118.061)
-		(width 0.2)
-		(layer "F.Cu")
-		(net 27)
-	)
-	(segment
-		(start 503.811002 118.061)
-		(end 502.750002 117)
-		(width 0.2)
-		(layer "F.Cu")
-		(net 27)
-	)
-	(segment
-		(start 514.395584 123)
-		(end 509.456584 118.061)
-		(width 0.2)
-		(layer "F.Cu")
-		(net 27)
-	)
-	(segment
-		(start 461.561 115.939)
-		(end 498.689003 115.939)
-		(width 0.2)
-		(layer "F.Cu")
-		(net 28)
-	)
-	(segment
-		(start 459.5 118)
-		(end 461.561 115.939)
-		(width 0.2)
-		(layer "F.Cu")
-		(net 28)
-	)
-	(segment
-		(start 498.689003 115.939)
-		(end 499.750003 117)
-		(width 0.2)
-		(layer "F.Cu")
-		(net 28)
-	)
-	(segment
-		(start 387.5 122.5)
-		(end 479.871526 122.5)
-		(width 0.2)
-		(layer "F.Cu")
-		(net 29)
-	)
-	(segment
-		(start 484.310526 118.061)
-		(end 495.689004 118.061)
-		(width 0.2)
-		(layer "F.Cu")
-		(net 29)
-	)
-	(segment
-		(start 479.871526 122.5)
-		(end 484.310526 118.061)
-		(width 0.2)
-		(layer "F.Cu")
-		(net 29)
-	)
-	(segment
-		(start 495.689004 118.061)
-		(end 496.750004 117)
-		(width 0.2)
-		(layer "F.Cu")
-		(net 29)
-	)
-	(segment
-		(start 386.894 121.644)
-		(end 386.894 123.356)
-		(width 0.2)
-		(layer "F.Cu")
-		(net 30)
-	)
-	(segment
-		(start 483.564 123.526)
-		(end 488.628 118.462)
-		(width 0.2)
-		(layer "F.Cu")
-		(net 30)
-	)
-	(segment
-		(start 387.064 123.526)
-		(end 483.564 123.526)
-		(width 0.2)
-		(layer "F.Cu")
-		(net 30)
-	)
-	(segment
-		(start 386.894 123.356)
-		(end 387.064 123.526)
-		(width 0.2)
-		(layer "F.Cu")
-		(net 30)
-	)
-	(segment
-		(start 315 118.5)
-		(end 318.144 121.644)
-		(width 0.2)
-		(layer "F.Cu")
-		(net 30)
-	)
-	(segment
-		(start 488.628 118.462)
-		(end 491.5 118.462)
-		(width 0.2)
-		(layer "F.Cu")
-		(net 30)
-	)
-	(segment
-		(start 318.144 121.644)
-		(end 386.894 121.644)
-		(width 0.2)
-		(layer "F.Cu")
-		(net 30)
 	)
 	(zone

Commit message: redid A
Routing:
- net /TEMP_8: track 0.00 -> 405.9 mm, vias 0 -> 2
- net /VOLT_8 +: track 0.00 -> 399.1 mm, vias 0 -> 1
- net /VOLT_7 +: track 0.00 -> 336.8 mm
- net /TEMP_7: track 0.00 -> 330.2 mm, vias 0 -> 2
- net /TEMP_6: track 0.00 -> 253.6 mm
- net /VOLT_6 +: track 0.00 -> 251.7 mm
- net /VOLT_5 +: track 0.00 -> 200.9 mm
- net /TEMP_5: track 0.00 -> 180.8 mm
- net /TEMP_1: track 0.00 -> 116.3 mm
- net /VOLT_4 +: track 0.00 -> 116.2 mm
- net /TEMP_4: track 0.00 -> 105.1 mm
- net /VOLT_1 +: track 0.00 -> 99.4 mm
- net /TEMP_2: track 0.00 -> 59.9 mm
- net /TEMP_3: track 0.00 -> 49.1 mm
- net /VOLT_3 +: track 0.00 -> 47.4 mm
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