File: Battery-SegmentPCB-B/Battery-SegmentPCB-B.kicad_pcb (KiCad board)
At the start: 2 copper layers, 556.2 x 27.7 mm, 10 parts, among them J11 Conn_01x04, J12 Conn_01x04, J13 Conn_01x04, J14 Conn_01x04, J15 Conn_01x04, J16 Conn_01x04, J17 Conn_01x04, J18 Conn_01x04, J19 Conn_01x09, J20 Conn_01x09

Commit message: FUCK I FORGOT B
Parts:
- added J1: Conn_01x01, MountingHole:MountingHole_3.2mm_M3_DIN965_Pad_TopOnly, F.Cu at (149.2, 110.6)
- added J10: Conn_01x09, footprints:CON_436500915_MOL, F.Cu at (484.2, 102.8)
- added J2: Conn_01x01, MountingHole:MountingHole_3.2mm_M3_DIN965_Pad_TopOnly, F.Cu at (149.2, 96.4)
- added J21: Conn_01x02, Connector_Molex:Molex_Nano-Fit_105309-xx02_1x02_P2.50mm_Vertical, F.Cu at (304.7, 101.5)
- added J22: Conn_01x02, Connector_Molex:Molex_Nano-Fit_105309-xx02_1x02_P2.50mm_Vertical, F.Cu at (373.9, 101.5)
- added J23: Conn_01x02, Connector_Molex:Molex_Nano-Fit_105309-xx02_1x02_P2.50mm_Vertical, F.Cu at (450.5, 102.0)
- added J24: Conn_01x02, Connector_Molex:Molex_Nano-Fit_105309-xx02_1x02_P2.50mm_Vertical, F.Cu at (520.0, 102.0)
- added J25: Conn_01x02, Connector_Molex:Molex_Nano-Fit_105309-xx02_1x02_P2.50mm_Vertical, F.Cu at (589.5, 102.0)
- added J26: Conn_01x02, Connector_Molex:Molex_Nano-Fit_105309-xx02_1x02_P2.50mm_Vertical, F.Cu at (658.9, 102.0)
- added J3: Conn_01x01, MountingHole:MountingHole_3.2mm_M3_DIN965_Pad_TopOnly, F.Cu at (221.1, 110.6)
- added J4: Conn_01x01, MountingHole:MountingHole_3.2mm_M3_DIN965_Pad_TopOnly, F.Cu at (221.1, 96.4)
- added J5: Conn_01x01, MountingHole:MountingHole_3.2mm_M3_DIN965_Pad_TopOnly, F.Cu at (292.9, 110.6)
- added J6: Conn_01x01, MountingHole:MountingHole_3.2mm_M3_DIN965_Pad_TopOnly, F.Cu at (292.9, 96.4)
- added J7: Conn_01x01, MountingHole:MountingHole_3.2mm_M3_DIN965_Pad_TopOnly, F.Cu at (364.7, 110.6)
- added J8: Conn_01x01, MountingHole:MountingHole_3.2mm_M3_DIN965_Pad_TopOnly, F.Cu at (364.7, 96.4)
- added J9: Conn_01x09, footprints:CON_436500915_MOL, F.Cu at (421.4, 102.7)
- J11, J12, J13, J14, J15, J16, J17, J18: value Conn_01x04 -> Conn_01x01; footprint footprints:CONN_S4B-PH-K-S_JST -> MountingHole:MountingHole_3.2mm_M3_DIN965_Pad_TopOnly; moved to F.Cu
- J19, J20: value Conn_01x09 -> Conn_01x02; footprint footprints:CON_436500915_MOL -> Connector_Molex:Molex_Nano-Fit_105309-xx02_1x02_P2.50mm_Vertical
- moved J14 371.4 mm to (508.4, 96.4), turned to 0 degrees
- moved J13 358.5 mm to (508.4, 110.6), turned to 0 degrees
- moved J19 277.0 mm to (172.4, 102.0), turned to 0 degrees
- moved J20 213.9 mm to (234.7, 101.2), turned to 0 degrees
- moved J12 156.5 mm to (436.5, 96.5), turned to 0 degrees
- moved J11 145.5 mm to (436.5, 110.6), turned to 0 degrees
- moved J18 108.5 mm to (652.0, 96.4), turned to 0 degrees
- moved J17 97.6 mm to (652.0, 110.6), turned to 0 degrees
- moved J15 38.2 mm to (580.2, 110.6), turned to 0 degrees
- moved J16 18.1 mm to (580.2, 96.5), turned to 0 degrees
Connections:
- J11 pad 1: /VOLT_1 - -> /VOLT_5 -
- J12 pad 1: /VOLT_2 - -> /VOLT1_5 +
- J13 pad 1: /VOLT_3 - -> /VOLT_6 -
- J14 pad 1: /VOLT_4 - -> /VOLT1_6 +
- J15 pad 1: /VOLT_5 - -> /VOLT_7 -
- J16 pad 1: /VOLT_6 - -> /VOLT1_7 +
- J17 pad 1: /VOLT_7 - -> /VOLT_8 -
- J18 pad 1: /VOLT_8 - -> /VOLT1_8 +
- J19 pad 2: /TEMP_2 -> /TEMP_GND
- J20 pad 1: /VOLT_1 - -> /TEMP_2
- J20 pad 2: /VOLT1_1 + -> /TEMP_GND
Routing:
- net /TEMP_GND: track 0.00 -> 494.3 mm
- net /TEMP_4: track 329.7 -> 41.4 mm
- net /TEMP_3: track 312.4 -> 114.0 mm
- net /VOLT1_4 +: track 331.1 -> 134.6 mm
- net /VOLT_1 -: track 155.0 -> 343.0 mm, vias 0 -> 2
- net /TEMP_8: track 79.0 -> 261.2 mm
- net /VOLT1_1 +: track 164.7 -> 336.7 mm
- net /VOLT1_8 +: track 66.3 -> 198.1 mm
- net /TEMP_5: track 154.3 -> 41.7 mm
- net /VOLT1_3 +: track 314.2 -> 202.2 mm
- net /TEMP_7: track 96.8 -> 187.8 mm
- net /VOLT1_2 +: track 181.0 -> 271.0 mm
- net /TEMP_1: track 162.8 -> 252.7 mm
- net /VOLT1_6 +: track 123.7 -> 47.8 mm
- net /VOLT1_5 +: track 141.4 -> 71.0 mm, vias 0 -> 2
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- removed copper zone on B.Cu, net /TEMP_GND
Other:
- board size 556.2 x 27.7 mm -> 522.7 x 21 mm
- board text added: "-"
- board text added: "1"
- board text added: "1+"
- board text added: "1-"
- board text added: "2"
- board text added: "2+"
- board text added: "2-"
- board text added: "3"
- board text added: "3+"
- board text added: "3-"
- board text added: "4"
- board text added: "4+"
- board text added: "4-"
- board text added: "5"
- board text added: "5+"
- board text added: "5-"
- board text added: "6"
- board text added: "6+"
- board text added: "6-"
- board text added: "7"
- board text added: "7+"
- board text added: "7-"
- board text added: "8"
- board text added: "8+"
- board text added: "8-"
- board text added: "Temperature Connector"
- board text added: "Voltage Connector"
