File: Battery-SegmentPCB-B/Battery-SegmentPCB-B.kicad_pcb (KiCad board)
At the start: 2 copper layers, 522.7 x 21 mm, 26 parts, among them J1 Conn_01x01, J10 Conn_01x09, J11 Conn_01x01, J12 Conn_01x01, J13 Conn_01x01, J14 Conn_01x01, J15 Conn_01x01, J16 Conn_01x01, J17 Conn_01x01, J18 Conn_01x01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

Commit message: b done
Parts:
- added F37: PTC Fuse, footprints:FUSC1810X100N, B.Cu at (154.8, 110.4)
- added F38: PTC Fuse, footprints:FUSC1810X100N, B.Cu at (226.3, 96.2)
- added F39: PTC Fuse, footprints:FUSC1810X100N, B.Cu at (298.1, 110.8)
- added F40: PTC Fuse, footprints:FUSC1810X100N, B.Cu at (370.1, 96.3)
- added F41: PTC Fuse, footprints:FUSC1810X100N, B.Cu at (647.0, 98.1)
- added F42: PTC Fuse, footprints:FUSC1810X100N, B.Cu at (574.1, 112.6)
- added F43: PTC Fuse, footprints:FUSC1810X100N, B.Cu at (513.8, 96.6)
- added F44: PTC Fuse, footprints:FUSC1810X100N, B.Cu at (441.8, 110.8)
- J1, J11, J12, J13, J14, J15, J16, J17, J18, J2, J3, J4, J5, J6, J7, J8: moved to B.Cu
- J19, J20, J21, J22, J23, J24, J25, J26: footprint Connector_Molex:Molex_Nano-Fit_105309-xx02_1x02_P2.50mm_Vertical -> UTSVT_Connectors:105313-2102
- moved J9 113.3 mm to (534.6, 108.0), turned to 180 degrees
- moved J10 74.5 mm to (558.6, 98.7)
- moved J24 27.6 mm to (493.4, 94.6), turned to -90 degrees
- moved J26 19.9 mm to (640.5, 94.6), turned to -90 degrees
- moved J15 14.1 mm to (580.2, 96.4)
- moved J11 14.1 mm to (436.5, 96.4)
- moved J2 14.1 mm to (149.2, 110.6)
- moved J5 14.1 mm to (292.9, 96.4)
- moved J6 14.1 mm to (292.9, 110.6)
- moved J1 14.1 mm to (149.2, 96.5)
- moved J12 14.1 mm to (436.5, 110.6)
- moved J16 14.1 mm to (580.2, 110.6)
- moved J22 10.3 mm to (381.5, 94.6), turned to -90 degrees
- moved J25 9.66 mm to (595.6, 94.6), turned to -90 degrees
- moved J23 8.06 mm to (453.6, 94.6), turned to -90 degrees
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Connections:
- J12 pad 1: /VOLT1_5 + -> Net-(J12-Pin_1)
- J14 pad 1: /VOLT1_6 + -> Net-(J14-Pin_1)
- J16 pad 1: /VOLT1_7 + -> Net-(J16-Pin_1)
- J18 pad 1: /VOLT1_8 + -> Net-(J18-Pin_1)
- J2 pad 1: /VOLT1_1 + -> Net-(J2-Pin_1)
- J4 pad 1: /VOLT1_2 + -> Net-(J4-Pin_1)
- J6 pad 1: /VOLT1_3 + -> Net-(J6-Pin_1)
- J8 pad 1: /VOLT1_4 + -> Net-(J8-Pin_1)
Routing:
- net /TEMP_8: track 261.2 -> 99.2 mm, vias 0 -> 1
- net /TEMP_4: track 41.4 -> 179.9 mm, vias 0 -> 3
- net /TEMP_3: track 114.0 -> 250.4 mm, vias 0 -> 1
- net /TEMP_7: track 187.8 -> 55.7 mm, vias 0 -> 1
- net /TEMP_2: track 187.4 -> 314.4 mm, vias 0 -> 1
- net /TEMP_1: track 252.7 -> 372.9 mm, vias 0 -> 1
- net /VOLT1_8 +: track 198.1 -> 117.6 mm, vias 0 -> 1
- net /VOLT1_1 +: track 336.7 -> 412.6 mm, vias 0 -> 1
- net /VOLT1_7 +: track 122.9 -> 47.1 mm, vias 0 -> 1
- net /VOLT_1 -: track 343.0 -> 413.4 mm, vias 2 -> 1
- net /VOLT1_2 +: track 271.0 -> 339.8 mm, vias 0 -> 2
- net /TEMP_5: track 41.7 -> 109.5 mm, vias 0 -> 3
- net /VOLT1_3 +: track 202.2 -> 259.8 mm, vias 0 -> 2
- net /VOLT1_4 +: track 134.6 -> 188.6 mm, vias 0 -> 2
- net /TEMP_6: track 114.8 -> 67.7 mm, vias 0 -> 4
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Other:
- outline, holes or cut-outs redrawn

Commit message: stuff
Parts:
- added G***: LHRs_LOGO, UTSVT_Logos:LHRs_LOGO, F.Cu at (595.8, 111.7)
- moved J19 0.84 mm to (174.5, 95.4)
- moved J21 0.51 mm to (308.4, 95.0)
- moved J20 0.42 mm to (236.3, 95.0)
- moved J22 0.39 mm to (381.6, 95.0)
- moved J23 0.34 mm to (453.6, 94.9)
- moved J24 0.27 mm to (493.5, 94.8)
- moved J26 0.17 mm to (640.5, 94.7)
- moved J25 0.15 mm to (595.6, 94.7)
Routing:
- net /TEMP_GND: track 511.8 -> 516.0 mm
- net /TEMP_1: track 372.9 -> 370.4 mm
- net /TEMP_4: track 179.9 -> 178.6 mm
Other:
- outline, holes or cut-outs redrawn
- board text added: "Battery B Segment Day Fixed"

Commit message: done?
Changed lines of the file:
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@@
-	)
-	(segment
-		(start 514.6411 95.549)
-		(end 552.723893 95.549)
-		(width 0.2)
-		(layer "F.Cu")
-		(net 2)
 	)
 	(segment
@@
 	)
 	(segment
-		(start 553.056093 95.549)
-		(end 555.488992 95.549)
-		(width 0.2)
-		(layer "F.Cu")
-		(net 2)
-	)
-	(segment
 		(start 158.649 99.324)
 		(end 488.6865 99.324)
@@
 	)
 	(segment
-		(start 514.3089 95.549)
-		(end 514.6411 95.549)
-		(width 0.2)
-		(layer "F.Cu")
-		(net 2)
-	)
-	(segment
 		(start 488.6865 99.324)
 		(end 489.4605 98.55)
@@
 	(segment
 		(start 513.976 95.549)
-		(end 514.3089 95.549)
-		(width 0.2)
-		(layer "F.Cu")
-		(net 2)
-	)
-	(segment
-		(start 552.723893 95.549)
-		(end 553.056093 95.549)
+		(end 555.488992 95.549)
 		(width 0.2)
 		(layer "F.Cu")
@@
 	)
 	(segment
-		(start 531.62722 107.927)
-		(end 531.95942 107.927)
-		(width 0.2)
-		(layer "F.Cu")
-		(net 6)
-	)
-	(segment
-		(start 535.661004 109.111)
-		(end 536.539003 109.111)
-		(width 0.2)
-		(layer "F.Cu")
-		(net 6)
-	)
-	(segment
-		(start 240.823 107.927)
-		(end 531.62722 107.927)
-		(width 0.2)
-		(layer "F.Cu")
-		(net 6)
-	)
-	(segment
 		(start 240.1 108.65)
 		(end 240.823 107.927)
@@
 	)
 	(segment
-		(start 531.95942 107.927)
+		(start 240.823 107.927)
 		(end 532.29162 107.927)
 		(width 0.2)
@@
 	(segment
 		(start 533.539004 109.111)
-		(end 535.661004 109.111)
-		(width 0.2)
-		(layer "F.Cu")
+		(end 536.539003 109.111)
+		(width 0.2)
+		(layer "F.Cu")

Commit message: seg B 4 layer
Parts:
- F37, F38, F39, F40, F41, F42, F43, F44: moved to F.Cu
- moved F42 8.94 mm to (579.5, 105.5)
- moved F38 6.80 mm to (222.0, 101.5)
- moved F44 6.79 mm to (437.5, 105.5)
- moved F39 6.73 mm to (294.0, 105.5)
- moved F37 6.53 mm to (150.0, 106.0)
- moved F40 6.52 mm to (365.5, 101.0)
- moved F43 6.46 mm to (509.0, 101.0)
- moved F41 5.30 mm to (651.0, 101.5)
- moved J9 1.05 mm to (534.6, 107.0)
- moved J10 0.79 mm to (558.6, 99.5)
Connections:
- net /VOLT1_1 + renamed /VOLT_1 +
- net /VOLT1_2 + renamed /VOLT_2 +
- net /VOLT1_3 + renamed /VOLT_3 +
- net /VOLT1_4 + renamed /VOLT_4 +
- net /VOLT1_5 + renamed /VOLT_5 +
- net /VOLT1_6 + renamed /VOLT_6 +
- net /VOLT1_7 + renamed /VOLT_7 +
- net /VOLT1_8 + renamed /VOLT_8 +
Routing:
- net /TEMP_GND: track 516.0 -> 0.00 mm, vias 2 -> 0
- net /VOLT_1 -: track 413.4 -> 0.00 mm, vias 1 -> 0
- net /VOLT_1 +: track 412.6 -> 0.00 mm, vias 1 -> 0
- net /TEMP_1: track 370.4 -> 0.00 mm, vias 1 -> 0
- net /VOLT_2 +: track 339.8 -> 0.00 mm, vias 2 -> 0
- net /TEMP_2: track 314.2 -> 0.00 mm, vias 1 -> 0
- net /VOLT_3 +: track 259.8 -> 0.00 mm, vias 2 -> 0
- net /TEMP_3: track 250.4 -> 0.00 mm, vias 1 -> 0
- net /VOLT_4 +: track 188.6 -> 0.00 mm, vias 2 -> 0
- net /TEMP_4: track 178.6 -> 0.00 mm, vias 3 -> 0
- net /VOLT_8 +: track 117.9 -> 0.00 mm, vias 1 -> 0
- net /VOLT_5 +: track 114.4 -> 0.00 mm, vias 2 -> 0
- net /TEMP_5: track 109.4 -> 0.00 mm, vias 3 -> 0
- net /TEMP_8: track 99.1 -> 0.00 mm, vias 1 -> 0
- net /TEMP_6: track 67.8 -> 0.00 mm, vias 4 -> 0
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- added copper zone on B.Cu, net /TEMP_GND
- added copper zone on In2.Cu, net /TEMP_GND
- added copper zone on F.Cu, net /VOLT_1 -
- added copper zone on In1.Cu, net /VOLT_1 -
Other:
- copper layers 2 -> 4

Commit message: redid b
Routing:
- net /VOLT_1 +: track 0.00 -> 413.2 mm
- net /TEMP_1: track 0.00 -> 365.5 mm
- net /VOLT_2 +: track 0.00 -> 335.4 mm, vias 0 -> 4
- net /TEMP_2: track 0.00 -> 307.6 mm
- net /VOLT_3 +: track 0.00 -> 263.1 mm
- net /TEMP_3: track 0.00 -> 239.7 mm
- net /VOLT_4 +: track 0.00 -> 186.2 mm
- net /TEMP_4: track 0.00 -> 168.5 mm
- net /VOLT_8 +: track 0.00 -> 120.0 mm
- net /VOLT_5 +: track 0.00 -> 107.6 mm
- net /TEMP_5: track 0.00 -> 99.5 mm
- net /TEMP_8: track 0.00 -> 92.0 mm
- net /TEMP_6: track 0.00 -> 61.2 mm
- net /TEMP_7: track 0.00 -> 49.5 mm
- net /VOLT_7 +: track 0.00 -> 44.2 mm
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