File: Battery-SegmentPCB-B/Battery-SegmentPCB-B.kicad_sch (KiCad schematic)
At the start: 26 parts, among them J1 Conn_01x01, J10 Conn_01x09, J11 Conn_01x01, J12 Conn_01x01, J13 Conn_01x01, J14 Conn_01x01, J15 Conn_01x01, J16 Conn_01x01, J17 Conn_01x01, J18 Conn_01x01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

Commit message: b done
Parts:
- added F37, F38, F39, F40, F41, F42, F43, F44: PTC Fuse, footprints:FUSC1810X100N, symbol Device:Polyfuse_Small
- J19, J20, J21, J22, J23, J24, J25, J26: footprint Connector_Molex:Molex_Nano-Fit_105309-xx02_1x02_P2.50mm_Vertical -> UTSVT_Connectors:105313-2102
Connections:
- net VOLT1_1 +: now also F37.1; no longer J2.1 (Pin_1)
- net VOLT1_2 +: now also F38.1; no longer J4.1 (Pin_1)
- net VOLT1_3 +: now also F39.1; no longer J6.1 (Pin_1)
- net VOLT1_4 +: now also F40.1; no longer J8.1 (Pin_1)
- net VOLT1_5 +: now also F44.1; no longer J12.1 (Pin_1)
- net VOLT1_6 +: now also F43.1; no longer J14.1 (Pin_1)
- net VOLT1_7 +: now also F42.1; no longer J16.1 (Pin_1)
- net VOLT1_8 +: now also F41.1; no longer J18.1 (Pin_1)
- new net: F40.2, J8.1 (Pin_1)
- new net: F37.2, J2.1 (Pin_1)
- new net: F38.2, J4.1 (Pin_1)
- new net: F39.2, J6.1 (Pin_1)
- new net: F41.2, J18.1 (Pin_1)
- new net: F43.2, J14.1 (Pin_1)
- new net: F44.2, J12.1 (Pin_1)
- new net: F42.2, J16.1 (Pin_1)
Other:
- moved on the sheet: J1, J2, J3, J4, J5, J6, J7, J8

Commit message: seg B 4 layer
Connections:
- net VOLT1_1 + renamed VOLT_1 +
- net VOLT1_2 + renamed VOLT_2 +
- net VOLT1_3 + renamed VOLT_3 +
- net VOLT1_4 + renamed VOLT_4 +
- net VOLT1_5 + renamed VOLT_5 +
- net VOLT1_6 + renamed VOLT_6 +
- net VOLT1_7 + renamed VOLT_7 +
- net VOLT1_8 + renamed VOLT_8 +
Changed lines of the file:
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@@
 		)
 	)
-	(label "VOLT1_7 +"
+	(label "VOLT_7 +"
 		(at 99.695 115.57 180)
 		(effects
@@
 		)
 	)
-	(label "VOLT1_4 +"
+	(label "VOLT_4 +"
 		(at 149.86 73.025 270)
 		(effects
@@
 		)
 	)
-	(label "VOLT1_6 +"
+	(label "VOLT_6 +"
 		(at 99.695 106.045 180)
 		(effects
@@
 		)
 	)
-	(label "VOLT1_7 +"
+	(label "VOLT_7 +"
 		(at 157.48 73.025 270)
 		(effects
@@
 		)
 	)
-	(label "VOLT1_1 +"
+	(label "VOLT_1 +"
 		(at 62.23 95.25 180)
 		(effects
@@
 		)
 	)
-	(label "VOLT1_8 +"
+	(label "VOLT_8 +"
 		(at 160.02 73.025 270)
 		(effects
@@
 		)
 	)
-	(label "VOLT1_2 +"
+	(label "VOLT_2 +"
 		(at 144.78 73.025 270)
 		(effects
@@
 		)
 	)
-	(label "VOLT1_3 +"
+	(label "VOLT_3 +"
 		(at 147.32 73.025 270)
 		(effects
@@
 		)
 	)
-	(label "VOLT1_4 +"
+	(label "VOLT_4 +"
 		(at 60.325 122.555 180)
 		(effects
@@
 		)
 	)
-	(label "VOLT1_3 +"
+	(label "VOLT_3 +"
 		(at 60.325 113.03 180)
 		(effects
@@
 		)
 	)
-	(label "VOLT1_1 +"
+	(label "VOLT_1 +"
 		(at 142.24 73.025 270)
 		(effects
@@
 		)
 	)
-	(label "VOLT1_8 +"
+	(label "VOLT_8 +"
 		(at 99.695 125.095 180)
 		(effects
@@
 		)
 	)
-	(label "VOLT1_5 +"
+	(label "VOLT_5 +"
 		(at 152.4 73.025 270)
 		(effects
@@
 		)
 	)
-	(label "VOLT1_5 +"
+	(label "VOLT_5 +"
 		(at 99.695 96.52 180)
 		(effects
@@
 		)
 	)
-	(label "VOLT1_6 +"
+	(label "VOLT_6 +"
 		(at 154.94 73.025 270)
 		(effects
@@
 		)
 	)
-	(label "VOLT1_2 +"
+	(label "VOLT_2 +"
 		(at 60.96 103.505 180)
 		(effects
